Commit message: Clean up iai_apartment

File: iai_apartment/mjcf/apartment/stl/apartment.urdf (robot description, URDF)
Before this commit: robot apartment, 126 links, 125 joints
Joints:
- joint cabinet10_drawer1_handle_joint: origin xyz=-0.24662336 -0.00124599 0.0172039 rpy=1.5707963267948966 0.0 0.0 -> xyz=-0.26662336 -0.00124599 0.0172039 rpy=1.5707963267948966 0.0 0.0
- joint cabinet10_drawer2_handle_joint: origin xyz=-0.24686237 -0.00397854 0.08541794 rpy=1.5707963267948966 0.0 0.0 -> xyz=-0.26686237 -0.00397854 0.08541794 rpy=1.5707963267948966 0.0 0.0
- joint cabinet10_drawer3_handle_joint: origin xyz=-0.24712164 -0.00402777 0.15116583 rpy=1.5707963267948966 0.0 0.0 -> xyz=-0.26712164 -0.00402777 0.15116583 rpy=1.5707963267948966 0.0 0.0
- joint cabinet11_drawer1_handle_joint: origin xyz=-0.24662336 -0.00124599 0.0172039 rpy=1.5707963267948966 0.0 0.0 -> xyz=-0.26662336 -0.00124599 0.0172039 rpy=1.5707963267948966 0.0 0.0
- joint cabinet11_drawer2_handle_joint: origin xyz=-0.24686237 -0.00397854 0.08541794 rpy=1.5707963267948966 0.0 0.0 -> xyz=-0.26686237 -0.00397854 0.08541794 rpy=1.5707963267948966 0.0 0.0
- joint cabinet11_drawer3_handle_joint: origin xyz=-0.24712164 -0.00402777 0.15116583 rpy=1.5707963267948966 0.0 0.0 -> xyz=-0.26712164 -0.00402777 0.15116583 rpy=1.5707963267948966 0.0 0.0
- joint cabinet1_door_handle_joint: origin xyz=-0.01559982 -0.46315559 -0.38983368 rpy=1.5707963267948966 0.0 0.0 -> xyz=-0.03598882 -0.46315559 -0.38983368 rpy=1.5707963267948966 0.0 0.0
- joint cabinet1_drawer1_handle_joint: origin xyz=-0.24792936 0.00091816 0.08401428 rpy=1.5707963267948966 0.0 0.0 -> xyz=-0.26831836 0.00091816 0.08401428 rpy=1.5707963267948966 0.0 0.0
- joint cabinet1_drawer2_handle_joint: origin xyz=-0.24909416 -0.00145845 0.150606 rpy=1.5707963267948966 0.0 0.0 -> xyz=-0.26948316 -0.00145845 0.150606 rpy=1.5707963267948966 0.0 0.0
- joint cabinet2_door_handle_joint: origin xyz=-0.00184994 -0.25886013 -0.10518866 rpy=1.5707963267948966 0.0 0.0 -> xyz=-0.02184994 -0.25886013 -0.10518866 rpy=1.5707963267948966 0.0 0.0
- joint cabinet4_door2_handle_joint: origin xyz=-0.04103859 -0.01415195 -0.13357088 rpy=1.5707963267948966 0.0 0.0 -> xyz=-0.06103859 -0.01415195 -0.13357088 rpy=1.5707963267948966 0.0 0.0
- joint cabinet5_drawer1_handle_joint: origin xyz=-0.24980946 0.00142363 0.01676949 rpy=1.5707963267948966 0.0 0.0 -> xyz=-0.26980946 0.00142363 0.01676949 rpy=1.5707963267948966 0.0 0.0
- joint cabinet5_drawer2_handle_joint: origin xyz=-0.2507106 0.00106413 0.08500843 rpy=1.5707963267948966 0.0 0.0 -> xyz=-0.2707106 0.00106413 0.08500843 rpy=1.5707963267948966 0.0 0.0
- joint cabinet5_drawer3_handle_joint: origin xyz=-0.24888186 0.00102875 0.15027037 rpy=1.5707963267948966 0.0 0.0 -> xyz=-0.26888186 0.00102875 0.15027037 rpy=1.5707963267948966 0.0 0.0
- joint cabinet6_drawer1_handle_joint: origin xyz=-0.24662336 -0.00124599 0.0172039 rpy=1.5707963267948966 0.0 0.0 -> xyz=-0.26662336 -0.00124599 0.0172039 rpy=1.5707963267948966 0.0 0.0
- joint cabinet6_drawer2_handle_joint: origin xyz=-0.24686237 -0.00397854 0.08541794 rpy=1.5707963267948966 0.0 0.0 -> xyz=-0.26686237 -0.00397854 0.08541794 rpy=1.5707963267948966 0.0 0.0
- joint cabinet6_drawer3_handle_joint: origin xyz=-0.24712164 -0.00402777 0.15116583 rpy=1.5707963267948966 0.0 0.0 -> xyz=-0.26712164 -0.00402777 0.15116583 rpy=1.5707963267948966 0.0 0.0
- joint cabinet9_drawer1_handle_joint: origin xyz=-0.24980946 0.00142363 0.01676949 rpy=1.5707963267948966 0.0 0.0 -> xyz=-0.26980946 0.00142363 0.01676949 rpy=1.5707963267948966 0.0 0.0
- joint cabinet9_drawer2_handle_joint: origin xyz=-0.2507106 0.00106413 0.08500843 rpy=1.5707963267948966 0.0 0.0 -> xyz=-0.2707106 0.00106413 0.08500843 rpy=1.5707963267948966 0.0 0.0
- joint cabinet9_drawer3_handle_joint: origin xyz=-0.24888186 0.00102875 0.15027037 rpy=1.5707963267948966 0.0 0.0 -> xyz=-0.26888186 0.00102875 0.15027037 rpy=1.5707963267948966 0.0 0.0
- joint dishwasher_front_handle_joint: origin xyz=-0.05493519 -0.67884796 0.0 rpy=0.0 0.0 0.0 -> xyz=-0.07493519 -0.67884796 0.0 rpy=0.0 0.0 0.0
- joint fridge_door1_handle_joint: origin xyz=-0.00799103 -0.46534321 -0.3616 rpy=1.5707963267948966 0.0 0.0 -> xyz=-0.02799103 -0.46534321 -0.3616 rpy=1.5707963267948966 0.0 0.0
- joint fridge_door2_handle_joint: origin xyz=0.00804657 -0.46538265 0.31786839 rpy=1.5707963267948966 0.0 0.0 -> xyz=0.02804657 -0.46538265 0.31786839 rpy=1.5707963267948966 0.0 0.0
- joint sink_drawer1_handle_joint: origin xyz=-0.24900223 0.00331339 0.35071747 rpy=1.5707963267948966 0.0 0.0 -> xyz=-0.26900223 0.00331339 0.35071747 rpy=1.5707963267948966 0.0 0.0
- joint window4_left_handle_joint: origin xyz=0.037617 0 -0.057755 rpy=0 0 0 -> xyz=0.067235 0 -0.057755 rpy=0 0 0
- joint window4_left_handle_rotation_joint: origin xyz=0.017383 -0.834107 0.0 rpy=0 0 0 -> xyz=0.01 -0.834107 0.0 rpy=0 0 0
- joint window4_right_handle_joint: origin xyz=0.037617 0 -0.057755 rpy=0 0 0 -> xyz=0.067235 0 -0.057755 rpy=0 0 0
- joint window4_right_handle_rotation_joint: origin xyz=0.017383 0.834107 0.0 rpy=0 0 0 -> xyz=0.01 0.834107 0.0 rpy=0 0 0

File: iai_apartment/urdf/apartment.urdf (robot description, URDF)
Before this commit: robot apartment, 126 links, 125 joints
Joints:
- joint cabinet10_drawer1_handle_joint: origin xyz=-0.24662336 -0.00124599 0.0172039 rpy=1.5707963267948966 0.0 0.0 -> xyz=-0.26662336 -0.00124599 0.0172039 rpy=1.5707963267948966 0.0 0.0
- joint cabinet10_drawer2_handle_joint: origin xyz=-0.24686237 -0.00397854 0.08541794 rpy=1.5707963267948966 0.0 0.0 -> xyz=-0.26686237 -0.00397854 0.08541794 rpy=1.5707963267948966 0.0 0.0
- joint cabinet10_drawer3_handle_joint: origin xyz=-0.24712164 -0.00402777 0.15116583 rpy=1.5707963267948966 0.0 0.0 -> xyz=-0.26712164 -0.00402777 0.15116583 rpy=1.5707963267948966 0.0 0.0
- joint cabinet11_drawer1_handle_joint: origin xyz=-0.24662336 -0.00124599 0.0172039 rpy=1.5707963267948966 0.0 0.0 -> xyz=-0.26662336 -0.00124599 0.0172039 rpy=1.5707963267948966 0.0 0.0
- joint cabinet11_drawer2_handle_joint: origin xyz=-0.24686237 -0.00397854 0.08541794 rpy=1.5707963267948966 0.0 0.0 -> xyz=-0.26686237 -0.00397854 0.08541794 rpy=1.5707963267948966 0.0 0.0
- joint cabinet11_drawer3_handle_joint: origin xyz=-0.24712164 -0.00402777 0.15116583 rpy=1.5707963267948966 0.0 0.0 -> xyz=-0.26712164 -0.00402777 0.15116583 rpy=1.5707963267948966 0.0 0.0
- joint cabinet1_door_handle_joint: origin xyz=-0.01559982 -0.46315559 -0.38983368 rpy=1.5707963267948966 0.0 0.0 -> xyz=-0.03598882 -0.46315559 -0.38983368 rpy=1.5707963267948966 0.0 0.0
- joint cabinet1_drawer1_handle_joint: origin xyz=-0.24792936 0.00091816 0.08401428 rpy=1.5707963267948966 0.0 0.0 -> xyz=-0.26831836 0.00091816 0.08401428 rpy=1.5707963267948966 0.0 0.0
- joint cabinet1_drawer2_handle_joint: origin xyz=-0.24909416 -0.00145845 0.150606 rpy=1.5707963267948966 0.0 0.0 -> xyz=-0.26948316 -0.00145845 0.150606 rpy=1.5707963267948966 0.0 0.0
- joint cabinet2_door_handle_joint: origin xyz=-0.00184994 -0.25886013 -0.10518866 rpy=1.5707963267948966 0.0 0.0 -> xyz=-0.02184994 -0.25886013 -0.10518866 rpy=1.5707963267948966 0.0 0.0
- joint cabinet4_door2_handle_joint: origin xyz=-0.04103859 -0.01415195 -0.13357088 rpy=1.5707963267948966 0.0 0.0 -> xyz=-0.06103859 -0.01415195 -0.13357088 rpy=1.5707963267948966 0.0 0.0
- joint cabinet5_drawer1_handle_joint: origin xyz=-0.24980946 0.00142363 0.01676949 rpy=1.5707963267948966 0.0 0.0 -> xyz=-0.26980946 0.00142363 0.01676949 rpy=1.5707963267948966 0.0 0.0
- joint cabinet5_drawer2_handle_joint: origin xyz=-0.2507106 0.00106413 0.08500843 rpy=1.5707963267948966 0.0 0.0 -> xyz=-0.2707106 0.00106413 0.08500843 rpy=1.5707963267948966 0.0 0.0
- joint cabinet5_drawer3_handle_joint: origin xyz=-0.24888186 0.00102875 0.15027037 rpy=1.5707963267948966 0.0 0.0 -> xyz=-0.26888186 0.00102875 0.15027037 rpy=1.5707963267948966 0.0 0.0
- joint cabinet6_drawer1_handle_joint: origin xyz=-0.24662336 -0.00124599 0.0172039 rpy=1.5707963267948966 0.0 0.0 -> xyz=-0.26662336 -0.00124599 0.0172039 rpy=1.5707963267948966 0.0 0.0
- joint cabinet6_drawer2_handle_joint: origin xyz=-0.24686237 -0.00397854 0.08541794 rpy=1.5707963267948966 0.0 0.0 -> xyz=-0.26686237 -0.00397854 0.08541794 rpy=1.5707963267948966 0.0 0.0
- joint cabinet6_drawer3_handle_joint: origin xyz=-0.24712164 -0.00402777 0.15116583 rpy=1.5707963267948966 0.0 0.0 -> xyz=-0.26712164 -0.00402777 0.15116583 rpy=1.5707963267948966 0.0 0.0
- joint cabinet9_drawer1_handle_joint: origin xyz=-0.24980946 0.00142363 0.01676949 rpy=1.5707963267948966 0.0 0.0 -> xyz=-0.26980946 0.00142363 0.01676949 rpy=1.5707963267948966 0.0 0.0
- joint cabinet9_drawer2_handle_joint: origin xyz=-0.2507106 0.00106413 0.08500843 rpy=1.5707963267948966 0.0 0.0 -> xyz=-0.2707106 0.00106413 0.08500843 rpy=1.5707963267948966 0.0 0.0
- joint cabinet9_drawer3_handle_joint: origin xyz=-0.24888186 0.00102875 0.15027037 rpy=1.5707963267948966 0.0 0.0 -> xyz=-0.26888186 0.00102875 0.15027037 rpy=1.5707963267948966 0.0 0.0
- joint dishwasher_front_handle_joint: origin xyz=-0.05493519 -0.67884796 0.0 rpy=0.0 0.0 0.0 -> xyz=-0.07493519 -0.67884796 0.0 rpy=0.0 0.0 0.0
- joint fridge_door1_handle_joint: origin xyz=-0.00799103 -0.46534321 -0.3616 rpy=1.5707963267948966 0.0 0.0 -> xyz=-0.02799103 -0.46534321 -0.3616 rpy=1.5707963267948966 0.0 0.0
- joint fridge_door2_handle_joint: origin xyz=0.00804657 -0.46538265 0.31786839 rpy=1.5707963267948966 0.0 0.0 -> xyz=0.02804657 -0.46538265 0.31786839 rpy=1.5707963267948966 0.0 0.0
- joint sink_drawer1_handle_joint: origin xyz=-0.24900223 0.00331339 0.35071747 rpy=1.5707963267948966 0.0 0.0 -> xyz=-0.26900223 0.00331339 0.35071747 rpy=1.5707963267948966 0.0 0.0
- joint window4_left_handle_joint: origin xyz=0.037617 0 -0.057755 rpy=0 0 0 -> xyz=0.067235 0 -0.057755 rpy=0 0 0
- joint window4_left_handle_rotation_joint: origin xyz=0.017383 -0.834107 0.0 rpy=0 0 0 -> xyz=0.01 -0.834107 0.0 rpy=0 0 0
- joint window4_right_handle_joint: origin xyz=0.037617 0 -0.057755 rpy=0 0 0 -> xyz=0.067235 0 -0.057755 rpy=0 0 0
- joint window4_right_handle_rotation_joint: origin xyz=0.017383 0.834107 0.0 rpy=0 0 0 -> xyz=0.01 0.834107 0.0 rpy=0 0 0

File: iai_apartment/urdf/envelope.xacro (robot description, xacro)
@@ -132,5 +132,5 @@
     </link>
     <joint name="window4_right_handle_rotation_joint" type="revolute">
-      <origin xyz="0.017383 0.834107 0.0" rpy="0 0 0" />
+      <origin xyz="0.01 0.834107 0.0" rpy="0 0 0" />
       <parent link="window4_right" />
       <child link="window4_right_handle_rotation" />
@@ -140,5 +140,5 @@
     <link name="window4_right_handle_rotation"/>
     <joint name="window4_right_handle_joint" type="fixed">
-      <origin xyz="0.037617 0 -0.057755" rpy="0 0 0" />
+      <origin xyz="0.067235 0 -0.057755" rpy="0 0 0" />
       <parent link="window4_right_handle_rotation" />
       <child link="window4_right_handle" />
@@ -151,5 +151,5 @@
       </visual>
       <collision>
-        <origin xyz="0 0 0.057814" rpy="0 ${pi/2} 0" />
+        <origin xyz="-0.029618 0 0.057814" rpy="0 ${pi/2} 0" />
         <geometry>
           <cylinder length="0.075236" radius="0.008" />
@@ -157,5 +157,5 @@
       </collision>
       <collision>
-        <origin xyz="0.029618 0 0" rpy="0 0 0" />
+        <origin xyz="0 0 0" rpy="0 0 0" />
         <geometry>
           <cylinder length="0.131626" radius="0.008" />
@@ -163,5 +163,5 @@
       </collision>
       <collision>
-        <origin xyz="0.011142 0 -0.057813" rpy="0 ${pi/2} 0" />
+        <origin xyz="-0.018476 0 -0.057813" rpy="0 ${pi/2} 0" />
         <geometry>
           <cylinder length="0.052952" radius="0.008" />
@@ -190,5 +190,5 @@
     </link>
     <joint name="window4_left_handle_rotation_joint" type="revolute">
-      <origin xyz="0.017383 -0.834107 0.0" rpy="0 0 0" />
+      <origin xyz="0.01 -0.834107 0.0" rpy="0 0 0" />
       <parent link="window4_left" />
       <child link="window4_left_handle_rotation" />
@@ -198,5 +198,5 @@
     <link name="window4_left_handle_rotation"/>
     <joint name="window4_left_handle_joint" type="fixed">
-      <origin xyz="0.037617 0 -0.057755" rpy="0 0 0" />
+      <origin xyz="0.067235 0 -0.057755" rpy="0 0 0" />
       <parent link="window4_left_handle_rotation" />
       <child link="window4_left_handle" />
@@ -209,5 +209,5 @@
       </visual>
       <collision>
-        <origin xyz="0 0 0.057814" rpy="0 ${pi/2} 0" />
+        <origin xyz="-0.029618 0 0.057814" rpy="0 ${pi/2} 0" />
         <geometry>
           <cylinder length="0.075236" radius="0.008" />
@@ -215,5 +215,5 @@
       </collision>
       <collision>
-        <origin xyz="0.029618 0 0" rpy="0 0 0" />
+        <origin xyz="0 0 0" rpy="0 0 0" />
         <geometry>
           <cylinder length="0.131626" radius="0.008" />
@@ -221,5 +221,5 @@
       </collision>
       <collision>
-        <origin xyz="0.011142 0 -0.057813" rpy="0 ${pi/2} 0" />
+        <origin xyz="-0.018476 0 -0.057813" rpy="0 ${pi/2} 0" />
         <geometry>
           <cylinder length="0.052952" radius="0.008" />
