Commit message: Clean up iai_apartment

File: iai_apartment/urdf/kitchen.xacro (robot description, xacro)
@@ -131,5 +131,5 @@
     </link>
     <joint name="cabinet1_door_handle_joint" type="fixed">
-      <origin xyz="-0.01559982 -0.46315559 -0.38983368" rpy="${pi/2} 0.0 0.0" />
+      <origin xyz="-0.03598882 -0.46315559 -0.38983368" rpy="${pi/2} 0.0 0.0" />
       <parent link="cabinet1_door" />
       <child link="cabinet1_door_handle" />
@@ -142,17 +142,17 @@
       </visual>
       <collision>
-        <origin xyz="-0.003891 0.0 0.08" />
-        <geometry>
-          <box size="0.02 0.013 0.013" />
-        </geometry>
-      </collision>
-      <collision>
-        <origin xyz="-0.003891 0.0 -0.08" />
-        <geometry>
-          <box size="0.02 0.013 0.013" />
-        </geometry>
-      </collision>
-      <collision>
-        <origin xyz="-0.0203895 0.0 0.0" />
+        <origin xyz="0.0164985 0.0 0.08" />
+        <geometry>
+          <box size="0.02 0.013 0.013" />
+        </geometry>
+      </collision>
+      <collision>
+        <origin xyz="0.0164985 0.0 -0.08" />
+        <geometry>
+          <box size="0.02 0.013 0.013" />
+        </geometry>
+      </collision>
+      <collision>
+        <origin xyz="0.0 0.0 0.0" />
         <geometry>
           <box size="0.013 0.013 0.173032" />
@@ -217,5 +217,5 @@
     </link>
     <joint name="cabinet1_drawer1_handle_joint" type="fixed">
-      <origin xyz="-0.24792936 0.00091816 0.08401428" rpy="${pi/2} 0.0 0.0" />
+      <origin xyz="-0.26831836 0.00091816 0.08401428" rpy="${pi/2} 0.0 0.0" />
       <parent link="cabinet1_drawer1" />
       <child link="cabinet1_drawer1_handle" />
@@ -228,17 +228,17 @@
       </visual>
       <collision>
-        <origin xyz="-0.003891 0.0 0.08" />
-        <geometry>
-          <box size="0.02 0.013 0.013" />
-        </geometry>
-      </collision>
-      <collision>
-        <origin xyz="-0.003891 0.0 -0.08" />
-        <geometry>
-          <box size="0.02 0.013 0.013" />
-        </geometry>
-      </collision>
-      <collision>
-        <origin xyz="-0.0203895 0.0 0.0" />
+        <origin xyz="0.0164985 0.0 0.08" />
+        <geometry>
+          <box size="0.02 0.013 0.013" />
+        </geometry>
+      </collision>
+      <collision>
+        <origin xyz="0.0164985 0.0 -0.08" />
+        <geometry>
+          <box size="0.02 0.013 0.013" />
+        </geometry>
+      </collision>
+      <collision>
+        <origin xyz="0.0 0.0 0.0" />
         <geometry>
           <box size="0.013 0.013 0.173032" />
@@ -303,5 +303,5 @@
     </link>
     <joint name="cabinet1_drawer2_handle_joint" type="fixed">
-      <origin xyz="-0.24909416 -0.00145845 0.150606" rpy="${pi/2} 0.0 0.0" />
+      <origin xyz="-0.26948316 -0.00145845 0.150606" rpy="${pi/2} 0.0 0.0" />
       <parent link="cabinet1_drawer2" />
       <child link="cabinet1_drawer2_handle" />
@@ -314,17 +314,17 @@
       </visual>
       <collision>
-        <origin xyz="-0.003891 0.0 0.08" />
-        <geometry>
-          <box size="0.02 0.013 0.013" />
-        </geometry>
-      </collision>
-      <collision>
-        <origin xyz="-0.003891 0.0 -0.08" />
-        <geometry>
-          <box size="0.02 0.013 0.013" />
-        </geometry>
-      </collision>
-      <collision>
-        <origin xyz="-0.0203895 0.0 0.0" />
+        <origin xyz="0.0164985 0.0 0.08" />
+        <geometry>
+          <box size="0.02 0.013 0.013" />
+        </geometry>
+      </collision>
+      <collision>
+        <origin xyz="0.0164985 0.0 -0.08" />
+        <geometry>
+          <box size="0.02 0.013 0.013" />
+        </geometry>
+      </collision>
+      <collision>
+        <origin xyz="0.0 0.0 0.0" />
         <geometry>
           <box size="0.013 0.013 0.173032" />
@@ -470,5 +470,5 @@
     </link>
     <joint name="cabinet2_door_handle_joint" type="fixed">
-      <origin xyz="-0.00184994 -0.25886013 -0.10518866" rpy="${pi/2} 0.0 0.0" />
+      <origin xyz="-0.02184994 -0.25886013 -0.10518866" rpy="${pi/2} 0.0 0.0" />
       <parent link="cabinet2_door" />
       <child link="cabinet2_door_handle" />
@@ -481,17 +481,17 @@
       </visual>
       <collision>
-        <origin xyz="-0.003891 0.0 0.08" />
-        <geometry>
-          <box size="0.02 0.013 0.013" />
-        </geometry>
-      </collision>
-      <collision>
-        <origin xyz="-0.003891 0.0 -0.08" />
-        <geometry>
-          <box size="0.02 0.013 0.013" />
-        </geometry>
-      </collision>
-      <collision>
-        <origin xyz="-0.0203895 0.0 0.0" />
+        <origin xyz="0.0164985 0.0 0.08" />
+        <geometry>
+          <box size="0.02 0.013 0.013" />
+        </geometry>
+      </collision>
+      <collision>
+        <origin xyz="0.0164985 0.0 -0.08" />
+        <geometry>
+          <box size="0.02 0.013 0.013" />
+        </geometry>
+      </collision>
+      <collision>
+        <origin xyz="0.0 0.0 0.0" />
         <geometry>
           <box size="0.013 0.013 0.173032" />
@@ -1037,5 +1037,5 @@
     </link>
     <joint name="fridge_door1_handle_joint" type="fixed">
-      <origin xyz="-0.00799103 -0.46534321 -0.3616" rpy="${pi/2} 0.0 0.0" />
+      <origin xyz="-0.02799103 -0.46534321 -0.3616" rpy="${pi/2} 0.0 0.0" />
       <parent link="fridge_door1" />
       <child link="fridge_door1_handle" />
@@ -1048,17 +1048,17 @@
       </visual>
       <collision>
-        <origin xyz="-0.003891 0.0 0.08" />
-        <geometry>
-          <box size="0.02 0.013 0.013" />
-        </geometry>
-      </collision>
-      <collision>
-        <origin xyz="-0.003891 0.0 -0.08" />
-        <geometry>
-          <box size="0.02 0.013 0.013" />
-        </geometry>
-      </collision>
-      <collision>
-        <origin xyz="-0.0203895 0.0 0.0" />
+        <origin xyz="0.0164985 0.0 0.08" />
+        <geometry>
+          <box size="0.02 0.013 0.013" />
+        </geometry>
+      </collision>
+      <collision>
+        <origin xyz="0.0164985 0.0 -0.08" />
+        <geometry>
+          <box size="0.02 0.013 0.013" />
+        </geometry>
+      </collision>
+      <collision>
+        <origin xyz="0.0 0.0 0.0" />
         <geometry>
           <box size="0.013 0.013 0.173032" />
@@ -1194,5 +1194,5 @@
     </link>
     <joint name="fridge_door2_handle_joint" type="fixed">
-      <origin xyz="0.00804657 -0.46538265 0.31786839" rpy="${pi/2} 0.0 0.0" />
+      <origin xyz="0.02804657 -0.46538265 0.31786839" rpy="${pi/2} 0.0 0.0" />
       <parent link="fridge_door2" />
       <child link="fridge_door2_handle" />
@@ -1205,17 +1205,17 @@
       </visual>
       <collision>
-        <origin xyz="-0.003891 0.0 0.08" />
-        <geometry>
-          <box size="0.02 0.013 0.013" />
-        </geometry>
-      </collision>
-      <collision>
-        <origin xyz="-0.003891 0.0 -0.08" />
-        <geometry>
-          <box size="0.02 0.013 0.013" />
-        </geometry>
-      </collision>
-      <collision>
-        <origin xyz="-0.0203895 0.0 0.0" />
+        <origin xyz="0.0164985 0.0 0.08" />
+        <geometry>
+          <box size="0.02 0.013 0.013" />
+        </geometry>
+      </collision>
+      <collision>
+        <origin xyz="0.0164985 0.0 -0.08" />
+        <geometry>
+          <box size="0.02 0.013 0.013" />
+        </geometry>
+      </collision>
+      <collision>
+        <origin xyz="0.0 0.0 0.0" />
         <geometry>
           <box size="0.013 0.013 0.173032" />
@@ -1673,5 +1673,5 @@
     </link>
     <joint name="cabinet4_door2_handle_joint" type="fixed">
-      <origin xyz="-0.04103859 -0.01415195 -0.13357088" rpy="${pi/2} 0.0 0.0" />
+      <origin xyz="-0.06103859 -0.01415195 -0.13357088" rpy="${pi/2} 0.0 0.0" />
       <parent link="cabinet4_door2" />
       <child link="cabinet4_door2_handle" />
@@ -1684,17 +1684,17 @@
       </visual>
       <collision>
-        <origin xyz="-0.003891 0.0 0.08" />
-        <geometry>
-          <box size="0.02 0.013 0.013" />
-        </geometry>
-      </collision>
-      <collision>
-        <origin xyz="-0.003891 0.0 -0.08" />
-        <geometry>
-          <box size="0.02 0.013 0.013" />
-        </geometry>
-      </collision>
-      <collision>
-        <origin xyz="-0.0203895 0.0 0.0" />
+        <origin xyz="0.0164985 0.0 0.08" />
+        <geometry>
+          <box size="0.02 0.013 0.013" />
+        </geometry>
+      </collision>
+      <collision>
+        <origin xyz="0.0164985 0.0 -0.08" />
+        <geometry>
+          <box size="0.02 0.013 0.013" />
+        </geometry>
+      </collision>
+      <collision>
+        <origin xyz="0.0 0.0 0.0" />
         <geometry>
           <box size="0.013 0.013 0.173032" />
@@ -1844,5 +1844,5 @@
     </link>
     <joint name="cabinet5_drawer1_handle_joint" type="fixed">
-      <origin xyz="-0.24980946 0.00142363 0.01676949" rpy="${pi/2} 0.0 0.0" />
+      <origin xyz="-0.26980946 0.00142363 0.01676949" rpy="${pi/2} 0.0 0.0" />
       <parent link="cabinet5_drawer1" />
       <child link="cabinet5_drawer1_handle" />
@@ -1855,17 +1855,17 @@
       </visual>
       <collision>
-        <origin xyz="-0.003891 0.0 0.08" />
-        <geometry>
-          <box size="0.02 0.013 0.013" />
-        </geometry>
-      </collision>
-      <collision>
-        <origin xyz="-0.003891 0.0 -0.08" />
-        <geometry>
-          <box size="0.02 0.013 0.013" />
-        </geometry>
-      </collision>
-      <collision>
-        <origin xyz="-0.0203895 0.0 0.0" />
+        <origin xyz="0.0164985 0.0 0.08" />
+        <geometry>
+          <box size="0.02 0.013 0.013" />
+        </geometry>
+      </collision>
+      <collision>
+        <origin xyz="0.0164985 0.0 -0.08" />
+        <geometry>
+          <box size="0.02 0.013 0.013" />
+        </geometry>
+      </collision>
+      <collision>
+        <origin xyz="0.0 0.0 0.0" />
         <geometry>
           <box size="0.013 0.013 0.173032" />
@@ -1930,5 +1930,5 @@
     </link>
     <joint name="cabinet5_drawer2_handle_joint" type="fixed">
-      <origin xyz="-0.2507106 0.00106413 0.08500843" rpy="${pi/2} 0.0 0.0" />
+      <origin xyz="-0.2707106 0.00106413 0.08500843" rpy="${pi/2} 0.0 0.0" />
       <parent link="cabinet5_drawer2" />
       <child link="cabinet5_drawer2_handle" />
@@ -1941,17 +1941,17 @@
       </visual>
       <collision>
-        <origin xyz="-0.003891 0.0 0.08" />
-        <geometry>
-          <box size="0.02 0.013 0.013" />
-        </geometry>
-      </collision>
-      <collision>
-        <origin xyz="-0.003891 0.0 -0.08" />
-        <geometry>
-          <box size="0.02 0.013 0.013" />
-        </geometry>
-      </collision>
-      <collision>
-        <origin xyz="-0.0203895 0.0 0.0" />
+        <origin xyz="0.0164985 0.0 0.08" />
+        <geometry>
+          <box size="0.02 0.013 0.013" />
+        </geometry>
+      </collision>
+      <collision>
+        <origin xyz="0.0164985 0.0 -0.08" />
+        <geometry>
+          <box size="0.02 0.013 0.013" />
+        </geometry>
+      </collision>
+      <collision>
+        <origin xyz="0.0 0.0 0.0" />
         <geometry>
           <box size="0.013 0.013 0.173032" />
@@ -2016,5 +2016,5 @@
     </link>
     <joint name="cabinet5_drawer3_handle_joint" type="fixed">
-      <origin xyz="-0.24888186 0.00102875 0.15027037" rpy="${pi/2} 0.0 0.0" />
+      <origin xyz="-0.26888186 0.00102875 0.15027037" rpy="${pi/2} 0.0 0.0" />
       <parent link="cabinet5_drawer3" />
       <child link="cabinet5_drawer3_handle" />
@@ -2027,17 +2027,17 @@
       </visual>
       <collision>
-        <origin xyz="-0.003891 0.0 0.08" />
-        <geometry>
-          <box size="0.02 0.013 0.013" />
-        </geometry>
-      </collision>
-      <collision>
-        <origin xyz="-0.003891 0.0 -0.08" />
-        <geometry>
-          <box size="0.02 0.013 0.013" />
-        </geometry>
-      </collision>
-      <collision>
-        <origin xyz="-0.0203895 0.0 0.0" />
+        <origin xyz="0.0164985 0.0 0.08" />
+        <geometry>
+          <box size="0.02 0.013 0.013" />
+        </geometry>
+      </collision>
+      <collision>
+        <origin xyz="0.0164985 0.0 -0.08" />
+        <geometry>
+          <box size="0.02 0.013 0.013" />
+        </geometry>
+      </collision>
+      <collision>
+        <origin xyz="0.0 0.0 0.0" />
         <geometry>
           <box size="0.013 0.013 0.173032" />
@@ -2133,5 +2133,5 @@
     </link>
     <joint name="cabinet6_drawer1_handle_joint" type="fixed">
-      <origin xyz="-0.24662336 -0.00124599 0.0172039" rpy="${pi/2} 0.0 0.0" />
+      <origin xyz="-0.26662336 -0.00124599 0.0172039" rpy="${pi/2} 0.0 0.0" />
       <parent link="cabinet6_drawer1" />
       <child link="cabinet6_drawer1_handle" />
@@ -2144,17 +2144,17 @@
       </visual>
       <collision>
-        <origin xyz="-0.003891 0.0 0.08" />
-        <geometry>
-          <box size="0.02 0.013 0.013" />
-        </geometry>
-      </collision>
-      <collision>
-        <origin xyz="-0.003891 0.0 -0.08" />
-        <geometry>
-          <box size="0.02 0.013 0.013" />
-        </geometry>
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
Commit message: Update apartment

File: iai_apartment/mjcf/apartment/stl/apartment.urdf (robot description, URDF)
Before this commit: robot apartment, 126 links, 125 joints
Links:
- removed link walls
- added link wall1; collision box size=18.76044 0.1285 3.0517; visual mesh filename=package://iai_apartment/meshes/visual/SM_Wall_01.dae
- added link wall2; collision box size=0.189552 4.9669 3.0517; visual mesh filename=package://iai_apartment/meshes/visual/SM_Wall_02.dae
- added link wall3; collision box size=8.2886 0.1285 3.0517; collision box size=8.47354 0.1285 3.0517
- added link wall4; collision box size=0.189552 4.9669 3.0517; visual mesh filename=package://iai_apartment/meshes/visual/SM_Wall_04.dae
Joints:
- removed joint walls_joint
- added joint wall1_joint: type fixed, parent envelope_root, child wall1, origin xyz=0 0 -0.2 rpy=0 0 0
- added joint wall2_joint: type fixed, parent envelope_root, child wall2, origin xyz=0 0 -0.2 rpy=0 0 0
- added joint wall3_joint: type fixed, parent envelope_root, child wall3, origin xyz=0 0 -0.2 rpy=0 0 0
- added joint wall4_joint: type fixed, parent envelope_root, child wall4, origin xyz=0 0 -0.2 rpy=0 0 0
- joint window4_frame_joint: parent walls -> envelope_root

File: iai_apartment/urdf/apartment.urdf (robot description, URDF)
Before this commit: robot apartment, 126 links, 125 joints
Links:
- removed link walls
- added link wall1; collision box size=18.76044 0.1285 3.0517; visual mesh filename=package://iai_apartment/meshes/visual/SM_Wall_01.dae
- added link wall2; collision box size=0.189552 4.9669 3.0517; visual mesh filename=package://iai_apartment/meshes/visual/SM_Wall_02.dae
- added link wall3; collision box size=8.2886 0.1285 3.0517; collision box size=8.47354 0.1285 3.0517
- added link wall4; collision box size=0.189552 4.9669 3.0517; visual mesh filename=package://iai_apartment/meshes/visual/SM_Wall_04.dae
Joints:
- removed joint walls_joint
- added joint wall1_joint: type fixed, parent envelope_root, child wall1, origin xyz=0 0 -0.2 rpy=0 0 0
- added joint wall2_joint: type fixed, parent envelope_root, child wall2, origin xyz=0 0 -0.2 rpy=0 0 0
- added joint wall3_joint: type fixed, parent envelope_root, child wall3, origin xyz=0 0 -0.2 rpy=0 0 0
- added joint wall4_joint: type fixed, parent envelope_root, child wall4, origin xyz=0 0 -0.2 rpy=0 0 0
- joint window4_frame_joint: parent walls -> envelope_root

File: iai_apartment/urdf/envelope.xacro (robot description, xacro)
@@ -8,13 +8,13 @@
     <link name="envelope_root" />
     <!-- things and stuff -->
-    <joint name="walls_joint" type="fixed">
-      <origin rpy="0 0 0" xyz="0 0 -0.2" />
-      <parent link="envelope_root" />
-      <child link="walls" />
-    </joint>
-    <link name="walls">
-      <visual>
-        <geometry>
-          <mesh filename="package://iai_apartment/meshes/visual/walls.dae" />
+    <joint name="wall1_joint" type="fixed">
+      <origin rpy="0 0 0" xyz="0 0 -0.2" />
+      <parent link="envelope_root" />
+      <child link="wall1" />
+    </joint>
+    <link name="wall1">
+      <visual>
+        <geometry>
+          <mesh filename="package://iai_apartment/meshes/visual/SM_Wall_01.dae" />
         </geometry>
       </visual>
@@ -25,4 +25,34 @@
         </geometry>
       </collision>
+    </link>
+    <joint name="wall2_joint" type="fixed">
+      <origin rpy="0 0 0" xyz="0 0 -0.2" />
+      <parent link="envelope_root" />
+      <child link="wall2" />
+    </joint>
+    <link name="wall2">
+      <visual>
+        <geometry>
+          <mesh filename="package://iai_apartment/meshes/visual/SM_Wall_02.dae" />
+        </geometry>
+      </visual>
+      <collision>
+        <origin xyz="-8.875 0.713447 1.73439" />
+        <geometry>
+          <box size="0.189552 4.9669 3.0517" />
+        </geometry>
+      </collision>
+    </link>
+    <joint name="wall3_joint" type="fixed">
+      <origin rpy="0 0 0" xyz="0 0 -0.2" />
+      <parent link="envelope_root" />
+      <child link="wall3" />
+    </joint>
+    <link name="wall3">
+      <visual>
+        <geometry>
+          <mesh filename="package://iai_apartment/meshes/visual/SM_Wall_03.dae" />
+        </geometry>
+      </visual>
       <collision>
         <origin xyz="-4.63823 3.27776 1.73439" />
@@ -37,12 +67,18 @@
         </geometry>
       </collision>
+    </link>
+    <joint name="wall4_joint" type="fixed">
+      <origin rpy="0 0 0" xyz="0 0 -0.2" />
+      <parent link="envelope_root" />
+      <child link="wall4" />
+    </joint>
+    <link name="wall4">
+      <visual>
+        <geometry>
+          <mesh filename="package://iai_apartment/meshes/visual/SM_Wall_04.dae" />
+        </geometry>
+      </visual>
       <collision>
         <origin xyz="9.98022 0.713447 1.73439" />
-        <geometry>
-          <box size="0.189552 4.9669 3.0517" />
-        </geometry>
-      </collision>
-      <collision>
-        <origin xyz="-8.875 0.713447 1.73439" />
         <geometry>
           <box size="0.189552 4.9669 3.0517" />
@@ -65,5 +101,5 @@
     <joint name="window4_frame_joint" type="fixed">
       <origin xyz="0.671098 3.37273 1.72145" rpy="0.0 0.0 ${-pi/2}"/>
-      <parent link="walls" />
+      <parent link="envelope_root" />
       <child link="window4_frame" />
     </joint>
