Commit message: Update apartment

File: iai_apartment/urdf/apartment.urdf (robot description, URDF)
Before this commit: robot apartment, 129 links, 128 joints
Joints:
- joint dishwasher_tray1_joint: origin xyz=0.19401426 0.00735926 0.22713593 rpy=0.0 0.0 0.0 -> xyz=0.22401426 0.00735926 0.22713593 rpy=0.0 0.0 0.0
- joint dishwasher_tray2_joint: origin xyz=0.17742002 0.00735798 0.40232784 rpy=0.0 0.0 0.0 -> xyz=0.20742002 0.00735798 0.40232784 rpy=0.0 0.0 0.0
- joint dishwasher_tray3_joint: origin xyz=0.19787212 0.01312525 0.61131351 rpy=0.0 0.0 0.0 -> xyz=0.22787212 0.01312525 0.61131351 rpy=0.0 0.0 0.0

File: iai_apartment/urdf/kitchen.xacro (robot description, xacro)
@@ -104,5 +104,4 @@
       </visual>
       <collision>
-        <origin xyz="0.0005 -0.009901 -0.361161 " />
         <geometry>
           <box size="0.534942 0.561938 0.015" />
@@ -2681,5 +2680,5 @@
     </link>
     <joint name="dishwasher_tray1_joint" type="prismatic">
-      <origin xyz="0.19401426 0.00735926 0.22713593" rpy="0.0 0.0 0.0" />
+      <origin xyz="0.22401426 0.00735926 0.22713593" rpy="0.0 0.0 0.0" />
       <parent link="dishwasher" />
       <child link="dishwasher_tray1" />
@@ -2725,5 +2724,5 @@
     </link>
     <joint name="dishwasher_tray2_joint" type="prismatic">
-      <origin xyz="0.17742002 0.00735798 0.40232784" rpy="0.0 0.0 0.0" />
+      <origin xyz="0.20742002 0.00735798 0.40232784" rpy="0.0 0.0 0.0" />
       <parent link="dishwasher" />
       <child link="dishwasher_tray2" />
@@ -2769,5 +2768,5 @@
     </link>
     <joint name="dishwasher_tray3_joint" type="prismatic">
-      <origin xyz="0.19787212 0.01312525 0.61131351" rpy="0.0 0.0 0.0" />
+      <origin xyz="0.22787212 0.01312525 0.61131351" rpy="0.0 0.0 0.0" />
       <parent link="dishwasher" />
       <child link="dishwasher_tray3" />

Commit message: Add damping for handle

File: iai_apartment/urdf/apartment.urdf (robot description, URDF)
Before this commit: robot apartment, 129 links, 128 joints
Joints:
- joint window4_frame_joint: origin xyz=0.671098 3.37273 1.72145 rpy=0.0 0.0 -1.5707963267948966 -> xyz=0.671098 3.37273 1.52145 rpy=0.0 0.0 -1.5707963267948966

File: iai_apartment/urdf/envelope.xacro (robot description, xacro)
@@ -100,5 +100,5 @@
     <!-- Window 4 -->
     <joint name="window4_frame_joint" type="fixed">
-      <origin xyz="0.671098 3.37273 1.72145" rpy="0.0 0.0 ${-pi/2}"/>
+      <origin xyz="0.671098 3.37273 1.52145" rpy="0.0 0.0 ${-pi/2}"/>
       <parent link="envelope_root" />
       <child link="window4_frame" />
