Commit message: Clean up

File: iai_apartment/urdf/apartment.urdf (robot description, URDF)
Before this commit: robot apartment, 129 links, 128 joints
Links:
- link armchair: geometry collision mesh filename=package://iai_apartment/meshes/stl/armchair.stl; visual mesh filename=package://iai_apartment/meshes/dae/armchair.dae
- link bedside_table: geometry collision box size=0.312 0.312 0.460; visual mesh filename=package://iai_apartment/meshes/dae/bedside_table.dae
- link cabinet1: geometry collision box size=0.008 0.561938 2.11178; collision box size=0.016 0.561938 0.064
- link cabinet10: geometry collision box size=0.008 0.369666 0.76582; collision box size=0.08 0.369666 0.016
- link cabinet10_drawer1: geometry collision box size=0.016 0.357644 0.085266; collision box size=0.019 0.397734 0.129986
- link cabinet10_drawer1_handle: geometry collision box size=0.013 0.013 0.173032; collision box size=0.02 0.013 0.013
- link cabinet10_drawer2: geometry collision box size=0.016 0.357644 0.168982; collision box size=0.019 0.397734 0.26275
- link cabinet10_drawer2_handle: geometry collision box size=0.013 0.013 0.173032; collision box size=0.02 0.013 0.013
- link cabinet10_drawer3: geometry collision box size=0.016 0.357644 0.16821; collision box size=0.019 0.397734 0.395734
- link cabinet10_drawer3_handle: geometry collision box size=0.013 0.013 0.173032; collision box size=0.02 0.013 0.013
- link cabinet11: geometry collision box size=0.008 0.86788 0.76582; collision box size=0.08 0.86788 0.016
- link cabinet11_drawer1: geometry collision box size=0.016 0.839576 0.085266; collision box size=0.019 0.896682 0.129986
- link cabinet11_drawer1_handle: geometry collision box size=0.013 0.013 0.173032; collision box size=0.02 0.013 0.013
- link cabinet11_drawer2: geometry collision box size=0.016 0.839576 0.168982; collision box size=0.019 0.896682 0.26275
- link cabinet11_drawer2_handle: geometry collision box size=0.013 0.013 0.173032; collision box size=0.02 0.013 0.013
- link cabinet11_drawer3: geometry collision box size=0.016 0.839576 0.16821; collision box size=0.019 0.896682 0.395734
- link cabinet11_drawer3_handle: geometry collision box size=0.013 0.013 0.173032; collision box size=0.02 0.013 0.013
- link cabinet1_door: geometry collision box size=0.019 0.596936 0.86681; visual mesh filename=package://iai_apartment/meshes/dae/SM_Kitchen_01_Door_01.dae
- link cabinet1_door_handle: geometry collision box size=0.013 0.013 0.173032; collision box size=0.02 0.013 0.013
- link cabinet1_drawer1: geometry collision box size=0.01865384 0.52364 0.16887; collision box size=0.019 0.596936 0.262972
- link cabinet1_drawer1_handle: geometry collision box size=0.013 0.013 0.173032; collision box size=0.02 0.013 0.013
- link cabinet1_drawer2: geometry collision box size=0.01865384 0.52364 0.1517224; collision box size=0.019 0.596936 0.39428
- link cabinet1_drawer2_handle: geometry collision box size=0.013 0.013 0.173032; collision box size=0.02 0.013 0.013
- link cabinet2: geometry collision box size=0.008 0.367764 2.09568; collision box size=0.014374 0.367764 0.063992
- link cabinet2_door: geometry collision box size=0.019 0.396958 2.12276; visual mesh filename=package://iai_apartment/meshes/dae/SM_Kitchen_02_Door.dae
- link cabinet2_door_handle: geometry collision box size=0.013 0.013 0.173032; collision box size=0.02 0.013 0.013
- link cabinet2_drawer1: geometry collision box size=0.016128 0.361962 0.10099; collision box size=0.017 0.361962 0.10099
- link cabinet2_drawer2: geometry collision box size=0.013796 0.361962 0.020298; collision box size=0.013796 0.361962 0.098
- link cabinet2_drawer3: geometry collision box size=0.013796 0.361962 0.020298; collision box size=0.013796 0.361962 0.098
- link cabinet2_drawer4: geometry collision box size=0.013796 0.361962 0.020298; collision box size=0.013796 0.361962 0.098
- link cabinet2_drawer5: geometry collision box size=0.013796 0.361962 0.020298; collision box size=0.013796 0.361962 0.098
- link cabinet2_drawer6: geometry collision box size=0.013796 0.361962 0.020298; collision box size=0.013796 0.361962 0.098
- link cabinet2_shelf: geometry collision box size=0.482948 0.367958 0.015; visual mesh filename=package://iai_apartment/meshes/dae/SM_Kitchen_02_Shelf.dae
- link cabinet3: geometry collision box size=0.016 0.147984 0.074692; collision box size=0.0209188 0.572134 0.06
- link cabinet4: geometry collision box size=0.01 0.967896 0.76582; collision box size=0.337962 0.967896 0.016
- link cabinet4_door1: geometry collision box size=0.019 0.994892 0.395736; visual mesh filename=package://iai_apartment/meshes/dae/SM_Kitchen_04_Door_01.dae
- link cabinet4_door2: geometry collision box size=0.019 0.994892 0.395736; visual mesh filename=package://iai_apartment/meshes/dae/SM_Kitchen_04_Door_02.dae
- link cabinet4_door2_handle: geometry collision box size=0.013 0.013 0.173032; collision box size=0.02 0.013 0.013
- link cabinet4_shelf1: geometry collision box size=0.307078 0.967896 0.008084; visual mesh filename=package://iai_apartment/meshes/dae/SM_Kitchen_04_Shelf.dae
- link cabinet4_shelf2: geometry collision box size=0.307078 0.967896 0.008084; visual mesh filename=package://iai_apartment/meshes/dae/SM_Kitchen_04_Shelf.dae
- link cabinet5: geometry collision box size=0.008 0.568134 0.76582; collision box size=0.08 0.568134 0.016
- link cabinet5_drawer1: geometry collision box size=0.016 0.539608 0.085266; collision box size=0.019 0.596936 0.129986
- link cabinet5_drawer1_handle: geometry collision box size=0.013 0.013 0.173032; collision box size=0.02 0.013 0.013
- link cabinet5_drawer2: geometry collision box size=0.016 0.539608 0.168982; collision box size=0.019 0.596936 0.26275
- link cabinet5_drawer2_handle: geometry collision box size=0.013 0.013 0.173032; collision box size=0.02 0.013 0.013
- link cabinet5_drawer3: geometry collision box size=0.016 0.539608 0.16821; collision box size=0.019 0.596936 0.395734
- link cabinet5_drawer3_handle: geometry collision box size=0.013 0.013 0.173032; collision box size=0.02 0.013 0.013
- link cabinet6: geometry collision box size=0.008 0.369666 0.76582; collision box size=0.08 0.369666 0.016
- link cabinet6_drawer1: geometry collision box size=0.016 0.357644 0.085266; collision box size=0.019 0.397734 0.129986
- link cabinet6_drawer1_handle: geometry collision box size=0.013 0.013 0.173032; collision box size=0.02 0.013 0.013
- link cabinet6_drawer2: geometry collision box size=0.016 0.357644 0.168982; collision box size=0.019 0.397734 0.26275
- link cabinet6_drawer2_handle: geometry collision box size=0.013 0.013 0.173032; collision box size=0.02 0.013 0.013
- link cabinet6_drawer3: geometry collision box size=0.016 0.357644 0.16821; collision box size=0.019 0.397734 0.395734
- link cabinet6_drawer3_handle: geometry collision box size=0.013 0.013 0.173032; collision box size=0.02 0.013 0.013
- link cabinet8: geometry collision box size=0.007888 0.568134 0.765818; collision box size=0.08 0.568134 0.016
- link cabinet9: geometry collision box size=0.007888 0.568134 0.765818; collision box size=0.08 0.568134 0.016
- link cabinet9_drawer1: geometry collision box size=0.016 0.539608 0.085266; collision box size=0.019 0.596936 0.129986
- link cabinet9_drawer1_handle: geometry collision box size=0.013 0.013 0.173032; collision box size=0.02 0.013 0.013
- link cabinet9_drawer2: geometry collision box size=0.016 0.539608 0.168982; collision box size=0.019 0.596936 0.26275
- link cabinet9_drawer2_handle: geometry collision box size=0.013 0.013 0.173032; collision box size=0.02 0.013 0.013
- link cabinet9_drawer3: geometry collision box size=0.016 0.539608 0.16821; collision box size=0.019 0.596936 0.395734
- link cabinet9_drawer3_handle: geometry collision box size=0.013 0.013 0.173032; collision box size=0.02 0.013 0.013
- link coffee_table: geometry collision box size=0.0673 0.4 0.32; collision box size=0.58 1.08 0.05954
- link coffee_table_drawer: geometry collision box size=0.0214 0.3486 0.2398; collision box size=0.0214 0.396 0.31569
- link counter_sink: geometry collision box size=0.02 0.404212 0.177388; collision box size=0.077992 0.404212 0.177388
- link counter_sink_stove: geometry collision box size=0.097634 3.17704 0.03; collision box size=0.475062 3.17704 0.03
- link counter_sink_tap: geometry collision cylinder length=0.024394 radius=0.022432; collision cylinder length=0.055994 radius=0.005
- link counter_wall: geometry collision box size=0.599 1.031064 0.026778; visual mesh filename=package://iai_apartment/meshes/dae/SM_Counter_Wall.dae
- link counter_watertab: geometry collision cylinder length=0.007636 radius=0.010966; collision cylinder length=0.077478 radius=0.022435
- link dishwasher: geometry collision box size=0.004826 0.597834 0.841796; collision box size=0.129522 0.015448 0.703882
- link dishwasher_front: geometry collision box size=0.018888 0.794358 0.609974; collision box size=0.03 0.679206 0.574938
- link dishwasher_front_handle: geometry collision box size=0.013 0.013 0.173032; collision box size=0.02 0.013 0.013
- link dishwasher_tray1: geometry collision box size=0.008578 0.538406 0.232972; collision box size=0.008578 0.538406 0.232972
- link dishwasher_tray2: geometry collision box size=0.008364 0.47464 0.175624; collision box size=0.008364 0.47464 0.175624
- link dishwasher_tray3: geometry collision box size=0.44 0.54 0.072; visual mesh filename=package://iai_apartment/meshes/dae/SM_Dishwasher_Tray_03.dae
- link fridge_base: geometry collision box size=0.01564 0.469566 0.929316; collision box size=0.116796 0.469566 0.56255
- link fridge_door1: geometry collision box size=0.018554 0.596492 1.336678; collision box size=0.025 0.553734 0.988894
- link fridge_door1_handle: geometry collision box size=0.013 0.013 0.173032; collision box size=0.02 0.013 0.013
- link fridge_door2: geometry collision box size=0.018554 0.596492 0.78594; collision box size=0.025 0.553734 0.622332
- link fridge_door2_handle: geometry collision box size=0.013 0.013 0.173032; collision box size=0.02 0.013 0.013
- link fridge_door_tray1: geometry collision box size=0.002 0.421854 0.095574; collision box size=0.002 0.421854 0.095574
- link fridge_door_tray2: geometry collision box size=0.002 0.421954 0.053802; collision box size=0.002 0.421954 0.053802
- link fridge_drawer1: geometry collision box size=0.002896 0.454234 0.095728; collision box size=0.004246 0.454234 0.164152
- link fridge_drawer2: geometry collision box size=0.002896 0.454234 0.064222; collision box size=0.004246 0.454234 0.137882
- link fridge_drawer3: geometry collision box size=0.002 0.408956 0.024924; collision box size=0.002 0.408956 0.11774
- link fridge_drawer4: geometry collision box size=0.002 0.408956 0.024924; collision box size=0.002 0.408956 0.08
- link fridge_drawer5: geometry collision box size=0.002 0.408808 0.024998; collision box size=0.002 0.408808 0.110706
- link fridge_egg_tray: geometry visual mesh filename=package://iai_apartment/meshes/dae/SM_Fridge_Egg_Tray.dae
- link fridge_shelf1: geometry collision box size=0.267982 0.468268 0.009088; visual mesh filename=package://iai_apartment/meshes/dae/SM_Fridge_Shelf.dae
- link fridge_shelf2: geometry collision box size=0.267982 0.468268 0.009088; visual mesh filename=package://iai_apartment/meshes/dae/SM_Fridge_Shelf.dae
- link island_cover1: geometry collision box size=0.01925 3.13566 0.90361; visual mesh filename=package://iai_apartment/meshes/dae/SM_Kitchen_Island_Cover_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
- link island_cover3: geometry collision box size=0.678888 0.02 0.90361; visual mesh filename=package://iai_apartment/meshes/dae/SM_Kitchen_Island_Cover_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
- link island_cover4: geometry collision box size=0.592148 0.019108 0.897013; visual mesh filename=package://iai_apartment/meshes/dae/SM_Kitchen_Island_Cover_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
- link island_cover5: geometry collision box size=0.678888 0.02 0.90361; visual mesh filename=package://iai_apartment/meshes/dae/SM_Kitchen_Island_Cover_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
- link kitchen1_base_board: geometry collision box size=0.019778 2.60316 0.1; visual mesh filename=package://iai_apartment/meshes/dae/SM_Kitchen_Base_Board_01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
- link kitchen2_base_board: geometry collision box size=0.02 3.11248 0.1; visual mesh filename=package://iai_apartment/meshes/dae/SM_Kitchen_Base_Board_02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
- link oven: geometry collision box size=0.074784 0.58989 0.586022; collision box size=0.545666 0.054902 0.586022
- link oven_door: geometry collision box size=0.471696 0.036998 0.590588; visual mesh filename=package://iai_apartment/meshes/dae/SM_Oven_Door.dae
- link sink_drawer1: geometry collision box size=0.016712 0.219652 0.34661; collision box size=0.016712 0.219652 0.34661
- link sink_drawer1_handle: geometry collision box size=0.013 0.013 0.173032; collision box size=0.02 0.013 0.013
- link sink_drawer2: geometry collision box size=0.016 0.557356 0.083; collision box size=0.017 0.064994 0.099322
- link sofa: geometry collision mesh filename=package://iai_apartment/meshes/stl/sofa.stl; visual mesh filename=package://iai_apartment/meshes/dae/sofa.dae
- link stove: geometry collision box size=0.516 0.795 0.004802; visual mesh filename=package://iai_apartment/meshes/dae/SM_Stove.dae
- link wall1: geometry collision box size=18.76044 0.1285 3.0517; visual mesh filename=package://iai_apartment/meshes/dae/SM_Wall_01.dae
- link wall2: geometry collision box size=0.189552 4.9669 3.0517; visual mesh filename=package://iai_apartment/meshes/dae/SM_Wall_02.dae
- link wall3: geometry collision box size=8.2886 0.1285 3.0517; collision box size=8.47354 0.1285 3.0517
- link wall4: geometry collision box size=0.189552 4.9669 3.0517; visual mesh filename=package://iai_apartment/meshes/dae/SM_Wall_04.dae
- link wardrobe: geometry collision box size=0.0367 1.0000 1.65; collision box size=0.0367 1.0000 1.65
- link wardrobe_door_left: geometry collision box size=0.012967 0.495438 1.64844; visual mesh filename=package://iai_apartment/meshes/dae/wardrobe_door_left.dae
- link wardrobe_door_left_handle: geometry collision box size=0.014486 0.015082 0.13; collision box size=0.033556 0.015082 0.014587
- link wardrobe_door_right: geometry collision box size=0.012967 0.495438 1.64844; visual mesh filename=package://iai_apartment/meshes/dae/wardrobe_door_right.dae
- link wardrobe_door_right_handle: geometry collision box size=0.014486 0.015082 0.13; collision box size=0.033556 0.015082 0.014587
- link window4_frame: geometry collision box size=0.02 0.146252 3.04322; collision box size=0.02 0.151148 3.04322
- link window4_left: geometry collision box size=0.02 0.86406 2.0631; visual mesh filename=package://iai_apartment/meshes/dae/SM_Window_Left.dae
- link window4_left_handle: geometry collision cylinder length=0.052952 radius=0.008; collision cylinder length=0.075236 radius=0.008
- link window4_right: geometry collision box size=0.02 0.843426 2.0631; visual mesh filename=package://iai_apartment/meshes/dae/SM_Window_Right.dae
- link window4_right_handle: geometry collision cylinder length=0.052952 radius=0.008; collision cylinder length=0.075236 radius=0.008
- link windows: geometry visual mesh filename=package://iai_apartment/meshes/dae/windows_without_4.dae

File: iai_apartment/urdf/envelope.xacro (robot description, xacro)
@@ -16,5 +16,5 @@
       <visual>
         <geometry>
-          <mesh filename="package://iai_apartment/meshes/visual/SM_Wall_01.dae" />
+          <mesh filename="package://iai_apartment/meshes/dae/SM_Wall_01.dae" />
         </geometry>
       </visual>
@@ -34,5 +34,5 @@
       <visual>
         <geometry>
-          <mesh filename="package://iai_apartment/meshes/visual/SM_Wall_02.dae" />
+          <mesh filename="package://iai_apartment/meshes/dae/SM_Wall_02.dae" />
         </geometry>
       </visual>
@@ -52,5 +52,5 @@
       <visual>
         <geometry>
-          <mesh filename="package://iai_apartment/meshes/visual/SM_Wall_03.dae" />
+          <mesh filename="package://iai_apartment/meshes/dae/SM_Wall_03.dae" />
         </geometry>
       </visual>
@@ -76,5 +76,5 @@
       <visual>
         <geometry>
-          <mesh filename="package://iai_apartment/meshes/visual/SM_Wall_04.dae" />
+          <mesh filename="package://iai_apartment/meshes/dae/SM_Wall_04.dae" />
         </geometry>
       </visual>
@@ -94,5 +94,5 @@
       <visual>
         <geometry>
-          <mesh filename="package://iai_apartment/meshes/visual/windows_without_4.dae" />
+          <mesh filename="package://iai_apartment/meshes/dae/windows_without_4.dae" />
         </geometry>
       </visual>
@@ -107,5 +107,5 @@
       <visual>
         <geometry>
-          <mesh filename="package://iai_apartment/meshes/visual/SM_Window_Frame.dae" />
+          <mesh filename="package://iai_apartment/meshes/dae/SM_Window_Frame.dae" />
         </geometry>
       </visual>
@@ -157,5 +157,5 @@
       <visual>
         <geometry>
-          <mesh filename="package://iai_apartment/meshes/visual/SM_Window_Right.dae" />
+          <mesh filename="package://iai_apartment/meshes/dae/SM_Window_Right.dae" />
         </geometry>
       </visual>
@@ -183,5 +183,5 @@
       <visual>
         <geometry>
-          <mesh filename="package://iai_apartment/meshes/visual/SM_Window_Handle.dae" />
+          <mesh filename="package://iai_apartment/meshes/dae/SM_Window_Handle.dae" />
         </geometry>
       </visual>
@@ -215,5 +215,5 @@
       <visual>
         <geometry>
-          <mesh filename="package://iai_apartment/meshes/visual/SM_Window_Left.dae" />
+          <mesh filename="package://iai_apartment/meshes/dae/SM_Window_Left.dae" />
         </geometry>
       </visual>
@@ -241,5 +241,5 @@
       <visual>
         <geometry>
-          <mesh filename="package://iai_apartment/meshes/visual/SM_Window_Handle.dae" />
+          <mesh filename="package://iai_apartment/meshes/dae/SM_Window_Handle.dae" />
         </geometry>
       </visual>

File: iai_apartment/urdf/furnitures.xacro (robot description, xacro)
@@ -15,5 +15,5 @@
       <visual>
         <geometry>
-          <mesh filename="package://iai_apartment/meshes/visual/wardrobe.dae" />
+          <mesh filename="package://iai_apartment/meshes/dae/wardrobe.dae" />
         </geometry>
       </visual>
@@ -119,5 +119,5 @@
       <visual>
         <geometry>
-          <mesh filename="package://iai_apartment/meshes/visual/wardrobe_door_left.dae" />
+          <mesh filename="package://iai_apartment/meshes/dae/wardrobe_door_left.dae" />
         </geometry>
       </visual>
@@ -137,5 +137,5 @@
       <visual>
         <geometry>
-          <mesh filename="package://iai_apartment/meshes/visual/wardrobe_door_handle.dae" />
+          <mesh filename="package://iai_apartment/meshes/dae/wardrobe_door_handle.dae" />
         </geometry>
       </visual>
@@ -169,5 +169,5 @@
       <visual>
         <geometry>
-          <mesh filename="package://iai_apartment/meshes/visual/wardrobe_door_right.dae" />
+          <mesh filename="package://iai_apartment/meshes/dae/wardrobe_door_right.dae" />
         </geometry>
       </visual>
@@ -187,5 +187,5 @@
       <visual>
         <geometry>
-          <mesh filename="package://iai_apartment/meshes/visual/wardrobe_door_handle.dae" />
+          <mesh filename="package://iai_apartment/meshes/dae/wardrobe_door_handle.dae" />
         </geometry>
       </visual>
@@ -217,10 +217,10 @@
       <visual>
         <geometry>
-          <mesh filename="package://iai_apartment/meshes/visual/armchair.dae" />
-        </geometry>
-      </visual>
-      <collision>
-        <geometry>
-          <mesh filename="package://iai_apartment/meshes/collision/armchair.stl" />
+          <mesh filename="package://iai_apartment/meshes/dae/armchair.dae" />
+        </geometry>
+      </visual>
+      <collision>
+        <geometry>
+          <mesh filename="package://iai_apartment/meshes/stf/armchair.stl" />
         </geometry>
       </collision>
@@ -234,10 +234,10 @@
       <visual>
         <geometry>
-          <mesh filename="package://iai_apartment/meshes/visual/sofa.dae" />
-        </geometry>
-      </visual>
-      <collision>
-        <geometry>
-          <mesh filename="package://iai_apartment/meshes/collision/sofa.stl" />
+          <mesh filename="package://iai_apartment/meshes/dae/sofa.dae" />
+        </geometry>
+      </visual>
+      <collision>
+        <geometry>
+          <mesh filename="package://iai_apartment/meshes/stf/sofa.stl" />
         </geometry>
       </collision>
@@ -251,5 +251,5 @@
       <visual>
         <geometry>
-          <mesh filename="package://iai_apartment/meshes/visual/coffee_table.dae" />
+          <mesh filename="package://iai_apartment/meshes/dae/coffee_table.dae" />
         </geometry>
       </visual>
@@ -300,5 +300,5 @@
       <visual>
         <geometry>
-          <mesh filename="package://iai_apartment/meshes/visual/coffee_table_drawer.dae" />
+          <mesh filename="package://iai_apartment/meshes/dae/coffee_table_drawer.dae" />
         </geometry>
       </visual>
@@ -342,5 +342,5 @@
       <visual>
         <geometry>
-          <mesh filename="package://iai_apartment/meshes/visual/bedside_table.dae" />
+          <mesh filename="package://iai_apartment/meshes/dae/bedside_table.dae" />
         </geometry>
       </visual>
