Commit message: Clean up

File: iai_apartment/urdf/kitchen.xacro (robot description, xacro)
@@ -24,5 +24,5 @@
       <visual>
         <geometry>
-          <mesh filename="package://iai_apartment/meshes/visual/SM_Kitchen_01_Base.dae" />
+          <mesh filename="package://iai_apartment/meshes/dae/SM_Kitchen_01_Base.dae" />
         </geometry>
       </visual>
@@ -119,5 +119,5 @@
       <visual>
         <geometry>
-          <mesh filename="package://iai_apartment/meshes/visual/SM_Kitchen_01_Door_01.dae" />
+          <mesh filename="package://iai_apartment/meshes/dae/SM_Kitchen_01_Door_01.dae" />
         </geometry>
       </visual>
@@ -137,5 +137,5 @@
       <visual>
         <geometry>
-          <mesh filename="package://iai_apartment/meshes/visual/SM_Kitchen_Handle.dae" />
+          <mesh filename="package://iai_apartment/meshes/dae/SM_Kitchen_Handle.dae" />
         </geometry>
       </visual>
@@ -169,5 +169,5 @@
       <visual>
         <geometry>
-          <mesh filename="package://iai_apartment/meshes/visual/SM_Kitchen_01_Drawer_01.dae" />
+          <mesh filename="package://iai_apartment/meshes/dae/SM_Kitchen_01_Drawer_01.dae" />
         </geometry>
       </visual>
@@ -223,5 +223,5 @@
       <visual>
         <geometry>
-          <mesh filename="package://iai_apartment/meshes/visual/SM_Kitchen_Handle.dae" />
+          <mesh filename="package://iai_apartment/meshes/dae/SM_Kitchen_Handle.dae" />
         </geometry>
       </visual>
@@ -255,5 +255,5 @@
       <visual>
         <geometry>
-          <mesh filename="package://iai_apartment/meshes/visual/SM_Kitchen_01_Drawer_02.dae" />
+          <mesh filename="package://iai_apartment/meshes/dae/SM_Kitchen_01_Drawer_02.dae" />
         </geometry>
       </visual>
@@ -309,5 +309,5 @@
       <visual>
         <geometry>
-          <mesh filename="package://iai_apartment/meshes/visual/SM_Kitchen_Handle.dae" />
+          <mesh filename="package://iai_apartment/meshes/dae/SM_Kitchen_Handle.dae" />
         </geometry>
       </visual>
@@ -339,5 +339,5 @@
       <visual>
         <geometry>
-          <mesh filename="package://iai_apartment/meshes/visual/SM_Oven.dae" />
+          <mesh filename="package://iai_apartment/meshes/dae/SM_Oven.dae" />
         </geometry>
       </visual>
@@ -383,5 +383,5 @@
       <visual>
         <geometry>
-          <mesh filename="package://iai_apartment/meshes/visual/SM_Oven_Door.dae" />
+          <mesh filename="package://iai_apartment/meshes/dae/SM_Oven_Door.dae" />
         </geometry>
       </visual>
@@ -402,5 +402,5 @@
       <visual>
         <geometry>
-          <mesh filename="package://iai_apartment/meshes/visual/SM_Kitchen_02_Base.dae" />
+          <mesh filename="package://iai_apartment/meshes/dae/SM_Kitchen_02_Base.dae" />
         </geometry>
       </visual>
@@ -458,5 +458,5 @@
       <visual>
         <geometry>
-          <mesh filename="package://iai_apartment/meshes/visual/SM_Kitchen_02_Door.dae" />
+          <mesh filename="package://iai_apartment/meshes/dae/SM_Kitchen_02_Door.dae" />
         </geometry>
       </visual>
@@ -476,5 +476,5 @@
       <visual>
         <geometry>
-          <mesh filename="package://iai_apartment/meshes/visual/SM_Kitchen_Handle.dae" />
+          <mesh filename="package://iai_apartment/meshes/dae/SM_Kitchen_Handle.dae" />
         </geometry>
       </visual>
@@ -506,5 +506,5 @@
       <visual>
         <geometry>
-          <mesh filename="package://iai_apartment/meshes/visual/SM_Kitchen_02_Shelf.dae" />
+          <mesh filename="package://iai_apartment/meshes/dae/SM_Kitchen_02_Shelf.dae" />
         </geometry>
       </visual>
@@ -526,5 +526,5 @@
       <visual>
         <geometry>
-          <mesh filename="package://iai_apartment/meshes/visual/SM_Kitchen_02_Drawer_01.dae" />
+          <mesh filename="package://iai_apartment/meshes/dae/SM_Kitchen_02_Drawer_01.dae" />
         </geometry>
       </visual>
@@ -570,5 +570,5 @@
       <visual>
         <geometry>
-          <mesh filename="package://iai_apartment/meshes/visual/SM_Kitchen_02_Drawer_02.dae" />
+          <mesh filename="package://iai_apartment/meshes/dae/SM_Kitchen_02_Drawer_02.dae" />
         </geometry>
       </visual>
@@ -644,5 +644,5 @@
       <visual>
         <geometry>
-          <mesh filename="package://iai_apartment/meshes/visual/SM_Kitchen_02_Drawer_02.dae" />
+          <mesh filename="package://iai_apartment/meshes/dae/SM_Kitchen_02_Drawer_02.dae" />
         </geometry>
       </visual>
@@ -718,5 +718,5 @@
       <visual>
         <geometry>
-          <mesh filename="package://iai_apartment/meshes/visual/SM_Kitchen_02_Drawer_02.dae" />
+          <mesh filename="package://iai_apartment/meshes/dae/SM_Kitchen_02_Drawer_02.dae" />
         </geometry>
       </visual>
@@ -792,5 +792,5 @@
       <visual>
         <geometry>
-          <mesh filename="package://iai_apartment/meshes/visual/SM_Kitchen_02_Drawer_02.dae" />
+          <mesh filename="package://iai_apartment/meshes/dae/SM_Kitchen_02_Drawer_02.dae" />
         </geometry>
       </visual>
@@ -866,5 +866,5 @@
       <visual>
         <geometry>
-          <mesh filename="package://iai_apartment/meshes/visual/SM_Kitchen_02_Drawer_02.dae" />
+          <mesh filename="package://iai_apartment/meshes/dae/SM_Kitchen_02_Drawer_02.dae" />
         </geometry>
       </visual>
@@ -939,5 +939,5 @@
       <visual>
         <geometry>
-          <mesh filename="package://iai_apartment/meshes/visual/SM_Kitchen_03_Fridge.dae" />
+          <mesh filename="package://iai_apartment/meshes/dae/SM_Kitchen_03_Fridge.dae" />
         </geometry>
       </visual>
@@ -1019,5 +1019,5 @@
       <visual>
         <geometry>
-          <mesh filename="package://iai_apartment/meshes/visual/SM_Fridge_Door_01.dae" />
+          <mesh filename="package://iai_apartment/meshes/dae/SM_Fridge_Door_01.dae" />
         </geometry>
       </visual>
@@ -1043,5 +1043,5 @@
       <visual>
         <geometry>
-          <mesh filename="package://iai_apartment/meshes/visual/SM_Kitchen_Handle.dae" />
+          <mesh filename="package://iai_apartment/meshes/dae/SM_Kitchen_Handle.dae" />
         </geometry>
       </visual>
@@ -1073,5 +1073,5 @@
       <visual>
         <geometry>
-          <mesh filename="package://iai_apartment/meshes/visual/SM_Fridge_Door_Tray_01.dae" />
+          <mesh filename="package://iai_apartment/meshes/dae/SM_Fridge_Door_Tray_01.dae" />
         </geometry>
       </visual>
@@ -1115,5 +1115,5 @@
       <visual>
         <geometry>
-          <mesh filename="package://iai_apartment/meshes/visual/SM_Fridge_Door_Tray_02.dae" />
+          <mesh filename="package://iai_apartment/meshes/dae/SM_Fridge_Door_Tray_02.dae" />
         </geometry>
       </visual>
@@ -1157,10 +1157,10 @@
       <visual>
         <geometry>
-          <mesh filename="package://iai_apartment/meshes/visual/SM_Fridge_Egg_Tray.dae" />
+          <mesh filename="package://iai_apartment/meshes/dae/SM_Fridge_Egg_Tray.dae" />
         </geometry>
       </visual>
       <!-- <collision>
         <geometry>
-          <mesh filename="package://iai_apartment/meshes/visual/SM_Fridge_Egg_Tray.stl" />
+          <mesh filename="package://iai_apartment/meshes/dae/SM_Fridge_Egg_Tray.stl" />
         </geometry>
       </collision> -->
@@ -1176,5 +1176,5 @@
       <visual>
         <geometry>
-          <mesh filename="package://iai_apartment/meshes/visual/SM_Fridge_Door_02.dae" />
+          <mesh filename="package://iai_apartment/meshes/dae/SM_Fridge_Door_02.dae" />
         </geometry>
       </visual>
@@ -1200,5 +1200,5 @@
       <visual>
         <geometry>
-          <mesh filename="package://iai_apartment/meshes/visual/SM_Kitchen_Handle.dae" />
+          <mesh filename="package://iai_apartment/meshes/dae/SM_Kitchen_Handle.dae" />
         </geometry>
       </visual>
@@ -1230,5 +1230,5 @@
       <visual>
         <geometry>
-          <mesh filename="package://iai_apartment/meshes/visual/SM_Fridge_Base.dae" />
+          <mesh filename="package://iai_apartment/meshes/dae/SM_Fridge_Base.dae" />
         </geometry>
       </visual>
@@ -1308,5 +1308,5 @@
       <visual>
         <geometry>
-          <mesh filename="package://iai_apartment/meshes/visual/SM_Fridge_Shelf.dae" />
+          <mesh filename="package://iai_apartment/meshes/dae/SM_Fridge_Shelf.dae" />
         </geometry>
       </visual>
@@ -1326,5 +1326,5 @@
       <visual>
         <geometry>
-          <mesh filename="package://iai_apartment/meshes/visual/SM_Fridge_Shelf.dae" />
+          <mesh filename="package://iai_apartment/meshes/dae/SM_Fridge_Shelf.dae" />
         </geometry>
       </visual>
@@ -1346,5 +1346,5 @@
       <visual>
         <geometry>
-          <mesh filename="package://iai_apartment/meshes/visual/SM_Fridge_Drawer_01.dae" />
+          <mesh filename="package://iai_apartment/meshes/dae/SM_Fridge_Drawer_01.dae" />
         </geometry>
       </visual>
@@ -1396,5 +1396,5 @@
       <visual>
         <geometry>
-          <mesh filename="package://iai_apartment/meshes/visual/SM_Fridge_Drawer_02.dae" />
+          <mesh filename="package://iai_apartment/meshes/dae/SM_Fridge_Drawer_02.dae" />
         </geometry>
       </visual>
@@ -1446,5 +1446,5 @@
       <visual>
         <geometry>
-          <mesh filename="package://iai_apartment/meshes/visual/SM_Fridge_Drawer_03.dae" />
+          <mesh filename="package://iai_apartment/meshes/dae/SM_Fridge_Drawer_03.dae" />
         </geometry>
       </visual>
@@ -1496,5 +1496,5 @@
       <visual>
         <geometry>
-          <mesh filename="package://iai_apartment/meshes/visual/SM_Fridge_Drawer_04.dae" />
+          <mesh filename="package://iai_apartment/meshes/dae/SM_Fridge_Drawer_04.dae" />
         </geometry>
       </visual>
@@ -1546,5 +1546,5 @@
       <visual>
         <geometry>
-          <mesh filename="package://iai_apartment/meshes/visual/SM_Fridge_Drawer_05.dae" />
+          <mesh filename="package://iai_apartment/meshes/dae/SM_Fridge_Drawer_05.dae" />
         </geometry>
       </visual>
@@ -1595,5 +1595,5 @@
       <visual>
         <geometry>
-          <mesh filename="package://iai_apartment/meshes/visual/SM_Kitchen_04_Base.dae" />
+          <mesh filename="package://iai_apartment/meshes/dae/SM_Kitchen_04_Base.dae" />
         </geometry>
       </visual>
@@ -1643,5 +1643,5 @@
       <visual>
         <geometry>
-          <mesh filename="package://iai_apartment/meshes/visual/SM_Kitchen_04_Door_01.dae" />
+          <mesh filename="package://iai_apartment/meshes/dae/SM_Kitchen_04_Door_01.dae" />
         </geometry>
       </visual>
@@ -1661,5 +1661,5 @@
       <visual>
         <geometry>
-          <mesh filename="package://iai_apartment/meshes/visual/SM_Kitchen_04_Door_02.dae" />
+          <mesh filename="package://iai_apartment/meshes/dae/SM_Kitchen_04_Door_02.dae" />
         </geometry>
       </visual>
@@ -1679,5 +1679,5 @@
       <visual>
         <geometry>
-          <mesh filename="package://iai_apartment/meshes/visual/SM_Kitchen_Handle.dae" />
+          <mesh filename="package://iai_apartment/meshes/dae/SM_Kitchen_Handle.dae" />
         </geometry>
       </visual>
@@ -1709,5 +1709,5 @@
       <visual>
         <geometry>
-          <mesh filename="package://iai_apartment/meshes/visual/SM_Kitchen_04_Shelf.dae" />
+          <mesh filename="package://iai_apartment/meshes/dae/SM_Kitchen_04_Shelf.dae" />
         </geometry>
       </visual>
@@ -1727,5 +1727,5 @@
       <visual>
         <geometry>
-          <mesh filename="package://iai_apartment/meshes/visual/SM_Kitchen_04_Shelf.dae" />
+          <mesh filename="package://iai_apartment/meshes/dae/SM_Kitchen_04_Shelf.dae" />
         </geometry>
       </visual>
@@ -1746,5 +1746,5 @@
       <visual>
         <geometry>
-          <mesh filename="package://iai_apartment/meshes/visual/SM_Counter_Wall.dae" />
+          <mesh filename="package://iai_apartment/meshes/dae/SM_Counter_Wall.dae" />
         </geometry>
       </visual>
@@ -1764,5 +1764,5 @@
       <visual>
         <geometry>
-          <mesh filename="package://iai_apartment/meshes/visual/SM_Kitchen_05_Base.dae" />
+          <mesh filename="package://iai_apartment/meshes/dae/SM_Kitchen_05_Base.dae" />
         </geometry>
       </visual>
@@ -1808,5 +1808,5 @@
       <visual>
         <geometry>
-          <mesh filename="package://iai_apartment/meshes/visual/SM_Kitchen_05_Drawer_01.dae" />
+          <mesh filename="package://iai_apartment/meshes/dae/SM_Kitchen_05_Drawer_01.dae" />
         </geometry>
       </visual>
@@ -1850,5 +1850,5 @@
       <visual>
         <geometry>
-          <mesh filename="package://iai_apartment/meshes/visual/SM_Kitchen_Handle.dae" />
+          <mesh filename="package://iai_apartment/meshes/dae/SM_Kitchen_Handle.dae" />
         </geometry>
       </visual>
@@ -1882,5 +1882,5 @@
       <visual>
         <geometry>
-          <mesh filename="package://iai_apartment/meshes/visual/SM_Kitchen_05_Drawer_02.dae" />
+          <mesh filename="package://iai_apartment/meshes/dae/SM_Kitchen_05_Drawer_02.dae" />
         </geometry>
       </visual>
@@ -1936,5 +1936,5 @@
       <visual>
         <geometry>
-          <mesh filename="package://iai_apartment/meshes/visual/SM_Kitchen_Handle.dae" />
+          <mesh filename="package://iai_apartment/meshes/dae/SM_Kitchen_Handle.dae" />
         </geometry>
       </visual>
@@ -1968,5 +1968,5 @@
       <visual>
         <geometry>
-          <mesh filename="package://iai_apartment/meshes/visual/SM_Kitchen_05_Drawer_03.dae" />
+          <mesh filename="package://iai_apartment/meshes/dae/SM_Kitchen_05_Drawer_03.dae" />
         </geometry>
       </visual>
@@ -2022,5 +2022,5 @@
       <visual>
         <geometry>
-          <mesh filename="package://iai_apartment/meshes/visual/SM_Kitchen_Handle.dae" />
+          <mesh filename="package://iai_apartment/meshes/dae/SM_Kitchen_Handle.dae" />
         </geometry>
       </visual>
@@ -2053,5 +2053,5 @@
       <visual>
         <geometry>
-          <mesh filename="package://iai_apartment/meshes/visual/SM_Kitchen_06_Base.dae" />
+          <mesh filename="package://iai_apartment/meshes/dae/SM_Kitchen_06_Base.dae" />
         </geometry>
       </visual>
@@ -2097,5 +2097,5 @@
       <visual>
         <geometry>
-          <mesh filename="package://iai_apartment/meshes/visual/SM_Kitchen_06_Drawer_01.dae" />
+          <mesh filename="package://iai_apartment/meshes/dae/SM_Kitchen_06_Drawer_01.dae" />
         </geometry>
       </visual>
@@ -2139,5 +2139,5 @@
       <visual>
         <geometry>
-          <mesh filename="package://iai_apartment/meshes/visual/SM_Kitchen_Handle.dae" />
+          <mesh filename="package://iai_apartment/meshes/dae/SM_Kitchen_Handle.dae" />
         </geometry>
       </visual>
@@ -2171,5 +2171,5 @@
       <visual>
         <geometry>
-          <mesh filename="package://iai_apartment/meshes/visual/SM_Kitchen_06_Drawer_02.dae" />
+          <mesh filename="package://iai_apartment/meshes/dae/SM_Kitchen_06_Drawer_02.dae" />
         </geometry>
       </visual>
@@ -2225,5 +2225,5 @@
       <visual>
         <geometry>
-          <mesh filename="package://iai_apartment/meshes/visual/SM_Kitchen_Handle.dae" />
+          <mesh filename="package://iai_apartment/meshes/dae/SM_Kitchen_Handle.dae" />
         </geometry>
       </visual>
@@ -2257,5 +2257,5 @@
       <visual>
         <geometry>
-          <mesh filename="package://iai_apartment/meshes/visual/SM_Kitchen_06_Drawer_03.dae" />
+          <mesh filename="package://iai_apartment/meshes/dae/SM_Kitchen_06_Drawer_03.dae" />
         </geometry>
       </visual>
@@ -2311,5 +2311,5 @@
       <visual>
         <geometry>
-          <mesh filename="package://iai_apartment/meshes/visual/SM_Kitchen_Handle.dae" />
+          <mesh filename="package://iai_apartment/meshes/dae/SM_Kitchen_Handle.dae" />
         </geometry>
       </visual>
@@ -2347,5 +2347,5 @@
       <visual>
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