Commit message: Fix typo

File: iai_apartment/urdf/furnitures.xacro (robot description, xacro)
@@ -222,5 +222,5 @@
       <collision>
         <geometry>
-          <mesh filename="package://iai_apartment/meshes/stf/armchair.stl" />
+          <mesh filename="package://iai_apartment/meshes/stl/armchair.stl" />
         </geometry>
       </collision>
@@ -239,5 +239,5 @@
       <collision>
         <geometry>
-          <mesh filename="package://iai_apartment/meshes/stf/sofa.stl" />
+          <mesh filename="package://iai_apartment/meshes/stl/sofa.stl" />
         </geometry>
       </collision>
